Commit message: Add solutions to lab08 tasks

File: lab08_activity/urdf/lab08_camera_description.urdf.xacro (robot description, xacro)
@@ -3,7 +3,11 @@
        name="camera" >
   <!-- Include camera description (Hint: look at camera_model.urdf.xacro within the lab08_activity package) -->
-  <!-- TODO: INSERT CODE HERE -->
+  <xacro:include filename="$(find lab08_activity)/urdf/camera_model.xacro" />
   <link name="world" />
   <!-- Link camera with world joint -->
-  <!-- TODO: INSERT CODE HERE -->
+  <joint name="camera_world_joint" type="fixed">
+    <parent link="world" />
+    <child link = "camera_link" />
+    <origin xyz="1.9 0.25 1.675" rpy="0.0 ${pi/2.6} ${pi}" />
+  </joint>
 </robot>

File: lab08_activity/urdf/lab08_robot_description.urdf.xacro (robot description, xacro)
@@ -3,7 +3,11 @@
        name="ur5e" >
   <!-- Include ur5e description (HINT: look at ur5e.xacro within the ur_description package)-->
-  <!-- TODO: INSERT CODE HERE -->
+  <xacro:include filename="$(find ur_description)/urdf/ur5e.xacro" />
   <link name="world" />
-  <!-- Link robot with world joint -->
-  <!-- TODO: INSERT CODE HERE -->
+  <!-- Link ur5e with world joint -->
+  <joint name="ur5e_world_joint" type="fixed">
+    <parent link="world" />
+    <child link = "base_link" />
+    <origin xyz="0.8 0.0 0.675" rpy="0.0 0.0 0.0" />
+  </joint>
 </robot>
